Commit message: pixed orietation [yh]

File: ffw_description/urdf/ffw_sg2_rev1_follower/ffw_sg2_follower.urdf (robot description, URDF)
Before this commit: robot ffw_sg2_follower, 40 links, 39 joints
Links:
- added link eepoint_l
- added link eepoint_r
- link camera_l_link: geometry collision box size=0.023 0.042 0.042; visual mesh filename=file:///home/youngho/git/ai-worker/ffw_description/meshes/c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 scale=0.001 0.001 0.001
- link camera_r_link: geometry collision box size=0.023 0.042 0.042; visual mesh filename=file:///home/youngho/git/ai-worker/ffw_description/meshes/c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 scale=0.001 0.001 0.001
Joints:
- added joint eepoint_l_joint: type fixed, parent gripper_l_rh_p12_rn_base, child eepoint_l, origin xyz=0 0 0.11 rpy=0 0 0
- added joint eepoint_r_joint: type fixed, parent gripper_r_rh_p12_rn_base, child eepoint_r, origin xyz=0 0 0.11 rpy=0 0 0
